Commit message: [ROS] wip on sample URDF

File: practicals/7-servo-project-2/code/robot-arm.urdf (robot description, URDF)
Before this commit: robot roco_arm, 1 links, 0 joints
Links:
- added link first_segment; visual box size=0.6 0.1 0.2
- link base_link: geometry visual cylinder length=0.06 radius=0.1
Joints:
- added joint base_to_first: type fixed, parent base_link, child first_segment, origin xyz=0 0 0.06

Commit message: [ROS] completed the bits to control servo in sync with URDF

File: practicals/7-servo-project-2/code/robot-arm.urdf (robot description, URDF)
Before this commit: robot roco_arm, 2 links, 1 joints
Links:
- link first_segment: geometry visual box size=0.6 0.05 0.1
Joints:
- joint base_to_first: axis (none) -> 0 1 0; limit (none) -> lower=0 upper=3.14 effort=1000 velocity=0.5; origin xyz=0 0 0.06 -> xyz=0 0 0.03; type fixed -> revolute
